File: SuperPower-uC/SuperPower-uC-KiCad/charger.sch (KiCad schematic (older format))
At the start: 0 parts

Commit message: Actually saved the changes as well
Changed lines of the file:
@@
 Text HLabel 1300 1700 0    50   BiDi ~ 0
 VBAT
+Text HLabel 1300 1900 0    50   Input ~ 0
+SCL
+Text HLabel 1300 2000 0    50   BiDi ~ 0
+SDA
 $EndSCHEMATC
