File: SuperPower-uC/SuperPower-uC-KiCad/charger_io.sch (KiCad schematic (older format))
At the start: 0 parts

Commit message: Actually saved the changes as well
Changed lines of the file:
@@
 Text HLabel 1300 1350 0    50   Output ~ 0
 VOUT
+Text HLabel 1300 1650 0    50   Input ~ 0
+D+
+Text HLabel 1300 1750 0    50   Input ~ 0
+D-
 $EndSCHEMATC
