File: SuperPower-uC/SuperPower-uC-KiCad/mcu.sch (KiCad schematic (older format))
At the start: 0 parts

Commit message: Actually saved the changes as well
Changed lines of the file:
@@
 Text HLabel 1300 1000 0    50   Input ~ 0
 3v3_MCU
+Text HLabel 1300 1150 0    50   BiDi ~ 0
+SDA
+Text HLabel 1300 1300 0    50   Input ~ 0
+SCL
+Text HLabel 1300 1550 0    50   Input ~ 0
+D+
+Text HLabel 1300 1650 0    50   Input ~ 0
+D-
 $EndSCHEMATC
