File: SuperPower-uC/SuperPower-uC-KiCad/rtc_cut_off.sch (KiCad schematic (older format))
At the start: 0 parts

Commit message: Actually saved the changes as well
Changed lines of the file:
@@
 Text HLabel 1600 1500 0    50   BiDi ~ 0
 SDA
+Text HLabel 1600 1800 0    50   Input ~ 0
+VIN
+Text HLabel 1600 1950 0    50   Output ~ 0
+VOUT
 $EndSCHEMATC
