File: SuperPower-uC/lowcost/charger.sch (KiCad schematic (older format))
At the start: 0 parts

Commit message: int pins and charging module
added Interrupt pins to the main sheet and finished the charging module sub sheet (with charger, fuel Gauge and power on int)
Parts:
- added C2: 0.1u, symbol Device:C
- added C3: 1u, Capacitor_SMD:C_0603_1608Metric_Pad1.05x0.95mm_HandSolder, symbol Device:C
- added C4: 10u, Capacitor_SMD:C_0603_1608Metric_Pad1.05x0.95mm_HandSolder, symbol Device:C
- added D1: LED, LED_SMD:LED_0603_1608Metric_Pad1.05x0.95mm_HandSolder, symbol Device:LED
- added J2: Thermistor, symbol Connector:Conn_01x02_Male
- added Q1, Q2: AO3401A, Package_TO_SOT_SMD:SOT-23, symbol Transistor_FET:AO3401A
- added R2: 100, symbol Device:R
- added R3: 10k, symbol Device:R
- added R4: 1k, Resistor_SMD:R_0603_1608Metric_Pad1.05x0.95mm_HandSolder, symbol Device:R
- added R5: 1.8k, Resistor_SMD:R_0603_1608Metric_Pad1.05x0.95mm_HandSolder, symbol Device:R
- added R6: 180k, Resistor_SMD:R_0603_1608Metric_Pad1.05x0.95mm_HandSolder, symbol Device:R
- added R7: 1M, Resistor_SMD:R_0603_1608Metric_Pad1.05x0.95mm_HandSolder, symbol Device:R
- added U3: LC709203FQH, Package_DFN_QFN:WDFN-8-1EP_4x3mm_P0.65mm_EP2.4x1.8mm, symbol LC709203FQH:LC709203FQH
- added U4: TP4054, Package_TO_SOT_SMD:SOT-23-5_HandSoldering, symbol TP4054:TP4054
Connections:
- net labels added: CHARGE-DISABLE, GND, INT, VCHARGE
- net labels removed: VBUS_IN, VIN, VSOLAR_IN
- wire segments 0 -> 50

Commit message: added ftdi and some cleanup
Parts:
- C2: footprint (none) -> Capacitor_SMD:C_0603_1608Metric_Pad1.05x0.95mm_HandSolder; LCSC (none) -> C14858
- J2: footprint (none) -> Resistor_SMD:R_0603_1608Metric_Pad1.05x0.95mm_HandSolder; LCSC (none) -> C76589
- Q1, Q2: footprint Package_TO_SOT_SMD:SOT-23 -> Package_TO_SOT_SMD:SOT-23_Handsoldering; LCSC (none) -> C347476
- R2: footprint (none) -> Resistor_SMD:R_0603_1608Metric_Pad1.05x0.95mm_HandSolder; LCSC (none) -> C22775
- R3: footprint (none) -> Resistor_SMD:R_0603_1608Metric_Pad1.05x0.95mm_HandSolder; LCSC (none) -> C25804
- U3: LCSC C152311 -> C152311
- U4: LCSC C32574 -> C32574
Changed lines of the file:
@@
 F 0 "Q2" H 1600 4700 50  0000 C CNN
 F 1 "AO3401A" H 1700 4400 50  0000 C CNN
-F 2 "Package_TO_SOT_SMD:SOT-23" H 1600 4475 50  0001 L CIN
+F 2 "Package_TO_SOT_SMD:SOT-23_Handsoldering" H 1600 4475 50  0001 L CIN
 F 3 "http://www.aosmd.com/pdfs/datasheet/AO3401A.pdf" H 1400 4550 50  0001 L CNN
+F 4 "C347476" H 1400 4550 50  0001 C CNN "LCSC"
 	1    1400 4550
 	1    0    0    1
@@
 F 0 "Q1" V 3442 3200 50  0000 C CNN
 F 1 "AO3401A" V 3351 3200 50  0000 C CNN
-F 2 "Package_TO_SOT_SMD:SOT-23" H 3300 3125 50  0001 L CIN
+F 2 "Package_TO_SOT_SMD:SOT-23_Handsoldering" H 3300 3125 50  0001 L CIN
 F 3 "http://www.aosmd.com/pdfs/datasheet/AO3401A.pdf" H 3100 3200 50  0001 L CNN
+F 4 "C347476" V 3100 3200 50  0001 C CNN "LCSC"
 	1    3100 3200
 	0    1    -1   0
@@
 F 2 "Package_TO_SOT_SMD:SOT-23-5_HandSoldering" H 1750 2950 50  0001 C CNN
 F 3 "https://datasheet.lcsc.com/szlcsc/Nanjing-Extension-Microelectronics-TP4054_C32574.pdf" H 1750 3200 50  0001 C CNN
-F 4 " C32574" H 1750 3200 50  0001 C CNN "LCSC"
+F 4 "C32574" H 1750 3200 50  0001 C CNN "LCSC"
 	1    1750 3200
 	-1   0    0    1
@@
 F 0 "J2" H 1908 2431 50  0000 C CNN
 F 1 "Thermistor" H 1908 2340 50  0000 C CNN
-F 2 "" H 1800 2250 50  0001 C CNN
-F 3 "~" H 1800 2250 50  0001 C CNN
+F 2 "Resistor_SMD:R_0603_1608Metric_Pad1.05x0.95mm_HandSolder" H 1800 2250 50  0001 C CNN
+F 3 "https://datasheet.lcsc.com/szlcsc/TDK-NTCG163JF103FT1_C76589.pdf" H 1800 2250 50  0001 C CNN
+F 4 "C76589" H 1800 2250 50  0001 C CNN "LCSC"
 	1    1800 2250
 	1    0    0    -1
@@
 F 0 "C2" H 1200 1600 50  0000 L CNN
 F 1 "0.1u" H 1200 1400 50  0000 L CNN
-F 2 "" H 1238 1350 50  0001 C CNN
+F 2 "Capacitor_SMD:C_0603_1608Metric_Pad1.05x0.95mm_HandSolder" H 1238 1350 50  0001 C CNN
 F 3 "~" H 1200 1500 50  0001 C CNN
+F 4 "C14858" H 1200 1500 50  0001 C CNN "LCSC"
 	1    1200 1500
 	1    0    0    -1
@@
 F 0 "R3" H 2370 1946 50  0000 L CNN
 F 1 "10k" H 2370 1855 50  0000 L CNN
-F 2 "" V 2230 1900 50  0001 C CNN
+F 2 "Resistor_SMD:R_0603_1608Metric_Pad1.05x0.95mm_HandSolder" V 2230 1900 50  0001 C CNN
 F 3 "~" H 2300 1900 50  0001 C CNN
+F 4 "C25804" H 2300 1900 50  0001 C CNN "LCSC"
 	1    2300 1900
 	1    0    0    -1
@@
 F 0 "R2" H 2670 1946 50  0000 L CNN
 F 1 "100" H 2670 1855 50  0000 L CNN
-F 2 "" V 2530 1900 50  0001 C CNN
+F 2 "Resistor_SMD:R_0603_1608Metric_Pad1.05x0.95mm_HandSolder" V 2530 1900 50  0001 C CNN
 F 3 "~" H 2600 1900 50  0001 C CNN
+F 4 "C22775" H 2600 1900 50  0001 C CNN "LCSC"
 	1    2600 1900
 	1    0    0    -1
@@
 F 2 "Package_DFN_QFN:WDFN-8-1EP_4x3mm_P0.65mm_EP2.4x1.8mm" H 1900 1350 50  0001 C CNN
 F 3 "https://www.onsemi.com/pub/Collateral/LC709203F-D.PDF" H 1850 1650 50  0001 C CNN
-F 4 " C152311" H 1850 1600 50  0001 C CNN "LCSC"
+F 4 "C152311" H 1850 1600 50  0001 C CNN "LCSC"
 	1    1850 1600
 	1    0    0    -1

Commit message: fixed mentioned issues and swapped micro usb with usb c
Connections:
- wire segments 50 -> 53
Changed lines of the file:
@@
 VCHARGE
 Wire Wire Line
-	1450 1750 1350 1750
-Text HLabel 1350 1750 0    50   BiDi ~ 0
+	1450 1750 1400 1750
+Text HLabel 1150 1650 0    50   BiDi ~ 0
 VBAT
 Wire Wire Line
@@
 Text HLabel 2350 1450 2    50   Input ~ 0
 SCL
+Wire Wire Line
+	1400 1750 1400 1550
+Wire Wire Line
+	1400 1550 1450 1550
+Connection ~ 1450 1550
+Connection ~ 1200 1650
+Wire Wire Line
+	1200 1650 1150 1650
 $EndSCHEMATC

Commit message: swapped tp4054 with tp4056
Parts:
- removed U4: TP4054, Package_TO_SOT_SMD:SOT-23-5_HandSoldering, symbol TP4054:TP4054
- added D2: LED, LED_SMD:LED_0603_1608Metric_Pad1.05x0.95mm_HandSolder, symbol Device:LED
- added R10: 1k, Resistor_SMD:R_0603_1608Metric_Pad1.05x0.95mm_HandSolder, symbol Device:R
- added U4: TP4056, Package_SO:SOP-8_3.9x4.9mm_P1.27mm, symbol TP4056:TP4056
- D1: LCSC C72041 -> C2286
- R4: value 1k -> 1.8k; LCSC C21190 -> C4177
Connections:
- wire segments 53 -> 58
Other:
- moved on the sheet: C3, D1, Q1, R4, R5, R6
Changed lines of the file:
@@
 Connection ~ 1150 4550
 Wire Wire Line
-	2350 3200 2350 3250
-Wire Wire Line
-	2100 3200 2350 3200
-Wire Wire Line
-	1350 3100 1400 3100
-Connection ~ 1350 3100
-Wire Wire Line
-	1350 2950 1350 3100
-Wire Wire Line
-	1400 2950 1350 2950
-Wire Wire Line
-	2150 3300 2100 3300
-Wire Wire Line
-	2150 2950 2150 3300
-Wire Wire Line
-	2100 2950 2150 2950
-Wire Wire Line
-	1700 2950 1800 2950
-Wire Wire Line
-	1200 3600 1300 3600
-Connection ~ 1200 3600
-Wire Wire Line
-	1200 3600 1200 3650
-Wire Wire Line
-	1100 3600 1200 3600
-Wire Wire Line
-	1300 3300 1400 3300
-Wire Wire Line
-	1100 3100 1350 3100
-Connection ~ 1100 3100
-Wire Wire Line
-	1100 3100 1100 3300
-Wire Wire Line
-	1050 3100 1100 3100
-Wire Wire Line
-	2700 3100 2100 3100
-Connection ~ 2700 3100
-Wire Wire Line
-	2700 3450 2700 3100
-Wire Wire Line
-	2750 3450 2700 3450
-Wire Wire Line
-	2900 3100 2700 3100
-Wire Wire Line
-	3350 3100 3300 3100
-Connection ~ 3100 3450
-Wire Wire Line
-	3150 3450 3100 3450
-Wire Wire Line
-	3100 3450 3050 3450
-Wire Wire Line
-	3100 3400 3100 3450
-Text HLabel 3150 3450 2    50   Input ~ 0
+	1100 3800 1200 3800
+Connection ~ 1100 3800
+Wire Wire Line
+	1100 3800 1100 3850
+Wire Wire Line
+	1000 3800 1100 3800
+Wire Wire Line
+	3050 3700 2800 3700
+Text HLabel 3100 3400 2    50   Input ~ 0
 CHARGE-DISABLE
-Text HLabel 3350 3100 2    50   BiDi ~ 0
+Text HLabel 3050 3700 2    50   BiDi ~ 0
 VBAT
 $Comp
 L Transistor_FET:AO3401A Q1
 U 1 1 5F8021C7
-P 3100 3200
-F 0 "Q1" V 3442 3200 50  0000 C CNN
-F 1 "AO3401A" V 3351 3200 50  0000 C CNN
-F 2 "Package_TO_SOT_SMD:SOT-23_Handsoldering" H 3300 3125 50  0001 L CIN
-F 3 "http://www.aosmd.com/pdfs/datasheet/AO3401A.pdf" H 3100 3200 50  0001 L CNN
-F 4 "C347476" V 3100 3200 50  0001 C CNN "LCSC"
-	1    3100 3200
+P 4100 2650
+F 0 "Q1" V 4442 2650 50  0000 C CNN
+F 1 "AO3401A" V 4351 2650 50  0000 C CNN
+F 2 "Package_TO_SOT_SMD:SOT-23_Handsoldering" H 4300 2575 50  0001 L CIN
+F 3 "http://www.aosmd.com/pdfs/datasheet/AO3401A.pdf" H 4100 2650 50  0001 L CNN
+F 4 "C347476" V 4100 2650 50  0001 C CNN "LCSC"
+	1    4100 2650
 	0    1    -1   0
 $EndComp
@@
 L Device:C C3
 U 1 1 5F7FD127
-P 1100 3450
-F 0 "C3" H 1100 3550 50  0000 L CNN
-F 1 "1u" H 1100 3350 50  0000 L CNN
-F 2 "Capacitor_SMD:C_0603_1608Metric_Pad1.05x0.95mm_HandSolder" H 1138 3300 50  0001 C CNN
-F 3 "~" H 1100 3450 50  0001 C CNN
-F 4 "C15849" H 1100 3450 50  0001 C CNN "LCSC"
-	1    1100 3450
-	1    0    0    -1
-$EndComp
-$Comp
-L power:GND #PWR?
-U 1 1 5F7FA92C
-P 2350 3250
-F 0 "#PWR?" H 2350 3000 50  0001 C CNN
-F 1 "GND" H 2355 3077 50  0000 C CNN
-F 2 "" H 2350 3250 50  0001 C CNN
-F 3 "" H 2350 3250 50  0001 C CNN
-	1    2350 3250
+P 1000 3650
+F 0 "C3" H 1000 3750 50  0000 L CNN
+F 1 "1u" H 1000 3550 50  0000 L CNN
+F 2 "Capacitor_SMD:C_0603_1608Metric_Pad1.05x0.95mm_HandSolder" H 1038 3500 50  0001 C CNN
+F 3 "~" H 1000 3650 50  0001 C CNN
+F 4 "C15849" H 1000 3650 50  0001 C CNN "LCSC"
+	1    1000 3650
 	1    0    0    -1
 $EndComp
@@
 L power:GND #PWR?
 U 1 1 5F7F85B4
-P 1200 3650
-F 0 "#PWR?" H 1200 3400 50  0001 C CNN
-F 1 "GND" H 1205 3477 50  0000 C CNN
-F 2 "" H 1200 3650 50  0001 C CNN
-F 3 "" H 1200 3650 50  0001 C CNN
-	1    1200 3650
+P 1100 3850
+F 0 "#PWR?" H 1100 3600 50  0001 C CNN
+F 1 "GND" H 1105 3677 50  0000 C CNN
+F 2 "" H 1100 3850 50  0001 C CNN
+F 3 "" H 1100 3850 50  0001 C CNN
+	1    1100 3850
 	1    0    0    -1
 $EndComp
@@
 L Device:LED D1
 U 1 1 5F7F2CDA
-P 1950 2950
-F 0 "D1" H 2050 2850 50  0000 C CNN
-F 1 "LED" H 1900 2800 50  0000 C CNN
-F 2 "LED_SMD:LED_0603_1608Metric_Pad1.05x0.95mm_HandSolder" H 1950 2950 50  0001 C CNN
-F 3 "~" H 1950 2950 50  0001 C CNN
-F 4 "C72041" H 1950 2950 50  0001 C CNN "LCSC"
-	1    1950 2950
+P 1850 3050
+F 0 "D1" H 1950 2950 50  0000 C CNN
+F 1 "LED" H 1800 2900 50  0000 C CNN
+F 2 "LED_SMD:LED_0603_1608Metric_Pad1.05x0.95mm_HandSolder" H 1850 3050 50  0001 C CNN
+F 3 "~" H 1850 3050 50  0001 C CNN
+F 4 "C2286" H 1850 3050 50  0001 C CNN "LCSC"
+	1    1850 3050
 	-1   0    0    1
 $EndComp
@@
 L Device:R R6
 U 1 1 5F7F0EE3
-P 2900 3450
-F 0 "R6" V 2800 3500 50  0000 L CNN
-F 1 "180k" V 2800 3250 50  0000 L CNN
-F 2 "Resistor_SMD:R_0603_1608Metric_Pad1.05x0.95mm_HandSolder" V 2830 3450 50  0001 C CNN
-F 3 "~" H 2900 3450 50  0001 C CNN
-F 4 "C22827" H 2900 3450 50  0001 C CNN "LCSC"
-	1    2900 3450
-	0    -1   -1   0
+P 2800 3550
+F 0 "R6" V 2700 3600 50  0000 L CNN
+F 1 "180k" V 2700 3350 50  0000 L CNN
+F 2 "Resistor_SMD:R_0603_1608Metric_Pad1.05x0.95mm_HandSolder" V 2730 3550 50  0001 C CNN
+F 3 "~" H 2800 3550 50  0001 C CNN
+F 4 "C22827" H 2800 3550 50  0001 C CNN "LCSC"
+	1    2800 3550
+	-1   0    0    1
 $EndComp
 $Comp
 L Device:R R5
 U 1 1 5F7F0AC0
-P 1300 3450
-F 0 "R5" H 1370 3496 50  0000 L CNN
-F 1 "1.8k" H 1350 3300 50  0000 L CNN
-F 2 "Resistor_SMD:R_0603_1608Metric_Pad1.05x0.95mm_HandSolder" V 1230 3450 50  0001 C CNN
-F 3 "~" H 1300 3450 50  0001 C CNN
-F 4 "C4177" H 1300 3450 50  0001 C CNN "LCSC"
-	1    1300 3450
+P 1200 3650
+F 0 "R5" H 1270 3696 50  0000 L CNN
+F 1 "1.8k" H 1250 3550 50  0000 L CNN
+F 2 "Resistor_SMD:R_0603_1608Metric_Pad1.05x0.95mm_HandSolder" V 1130 3650 50  0001 C CNN
+F 3 "~" H 1200 3650 50  0001 C CNN
+F 4 "C4177" H 1200 3650 50  0001 C CNN "LCSC"
+	1    1200 3650
 	1    0    0    -1
 $EndComp
@@
 L Device:R R4
 U 1 1 5F7F0079
-P 1550 2950
-F 0 "R4" V 1650 3000 50  0000 L CNN
-F 1 "1k" V 1650 2800 50  0000 L CNN
-F 2 "Resistor_SMD:R_0603_1608Metric_Pad1.05x0.95mm_HandSolder" V 1480 2950 50  0001 C CNN
-F 3 "~" H 1550 2950 50  0001 C CNN
-F 4 "C21190" V 1550 2950 50  0001 C CNN "LCSC"
-	1    1550 2950
-	0    -1   -1   0
-$EndComp
-$Comp
-L TP4054:TP4054 U4
-U 1 1 5F7EF510
-P 1750 3200
-F 0 "U4" H 1950 3450 50  0000 C CNN
-F 1 "TP4054" H 1650 3450 50  0000 C CNN
-F 2 "Package_TO_SOT_SMD:SOT-23-5_HandSoldering" H 1750 2950 50  0001 C CNN
-F 3 "https://datasheet.lcsc.com/szlcsc/Nanjing-Extension-Microelectronics-TP4054_C32574.pdf" H 1750 3200 50  0001 C CNN
-F 4 "C32574" H 1750 3200 50  0001 C CNN "LCSC"
-	1    1750 3200
-	-1   0    0    1
-$EndComp
-Text HLabel 1050 3100 0    50   Input ~ 0
+P 2450 3200
+F 0 "R4" V 2550 3250 50  0000 L CNN
+F 1 "1.8k" V 2550 3050 50  0000 L CNN
+F 2 "Resistor_SMD:R_0603_1608Metric_Pad1.05x0.95mm_HandSolder" V 2380 3200 50  0001 C CNN
+F 3 "~" H 2450 3200 50  0001 C CNN
+F 4 "C4177" V 2450 3200 50  0001 C CNN "LCSC"
+	1    2450 3200
+	1    0    0    -1
+$EndComp
+Text HLabel 900  3300 0    50   Input ~ 0
 VCHARGE
 Wire Wire Line
@@
 Wire Wire Line
 	1200 1650 1150 1650
+$Comp
+L TP4056:TP4056 U4
+U 1 1 5F7DFABD
+P 1900 3500
+F 0 "U4" H 2100 3700 50  0000 C CNN
+F 1 "TP4056" H 1800 3700 50  0000 C CNN
+F 2 "Package_SO:SOP-8_3.9x4.9mm_P1.27mm" H 1900 3750 50  0001 C CNN
+F 3 "https://dlnmh9ip6v2uc.cloudfront.net/datasheets/Prototyping/TP4056.pdf" H 1900 3750 50  0001 C CNN
+F 4 "C16581" H 1950 3150 50  0001 C CNN "LCSC"
+	1    1900 3500
+	1    0    0    -1
+$EndComp
+$Comp
+L Device:LED D2
+U 1 1 5F7EC7D0
+P 2300 2900
+F 0 "D2" H 2400 2800 50  0000 C CNN
+F 1 "LED" H 2250 2750 50  0000 C CNN
+F 2 "LED_SMD:LED_0603_1608Metric_Pad1.05x0.95mm_HandSolder" H 2300 2900 50  0001 C CNN
+F 3 "~" H 2300 2900 50  0001 C CNN
+F 4 "C72041" H 2300 2900 50  0001 C CNN "LCSC"
+	1    2300 2900
+	-1   0    0    1
+$EndComp
+Wire Wire Line
+	900  3300 1000 3300
+Wire Wire Line
+	1400 3700 1500 3700
+Wire Wire Line
+	1500 3600 1450 3600
+Wire Wire Line
+	1450 3600 1450 3800
+Wire Wire Line
+	1450 3800 1200 3800
+Connection ~ 1200 3800
+Wire Wire Line
+	1400 3300 1400 3700
+Wire Wire Line
+	1200 3500 1500 3500
+Wire Wire Line
+	1500 3400 1450 3400
+Wire Wire Line
+	1450 3400 1450 3600
+Connection ~ 1450 3600
+Wire Wire Line
+	3100 3400 2800 3400
+$Comp
+L Device:R R10
+U 1 1 5F807B88
+P 2650 3200
+F 0 "R10" V 2750 3250 50  0000 L CNN
+F 1 "1k" V 2750 3050 50  0000 L CNN
+F 2 "Resistor_SMD:R_0603_1608Metric_Pad1.05x0.95mm_HandSolder" V 2580 3200 50  0001 C CNN
+F 3 "~" H 2650 3200 50  0001 C CNN
+F 4 "C21190" V 2650 3200 50  0001 C CNN "LCSC"
+	1    2650 3200
+	1    0    0    -1
+$EndComp
+Wire Wire Line
+	2450 3350 2450 3500
+Wire Wire Line
+	2450 3500 2300 3500
+Wire Wire Line
+	2300 3600 2650 3600
+Wire Wire Line
+	2650 3600 2650 3350
+Wire Wire Line
+	2000 3050 2450 3050
+Wire Wire Line
+	2450 2900 2650 2900
+Wire Wire Line
+	2650 2900 2650 3050
+Wire Wire Line
+	1700 3050 1400 3050
+Wire Wire Line
+	1400 3050 1400 3300
+Connection ~ 1400 3300
+Wire Wire Line
+	1400 3050 1400 2900
+Wire Wire Line
+	1400 2900 2150 2900
+Connection ~ 1400 3050
+Wire Wire Line
+	1000 3500 1000 3300
+Connection ~ 1000 3300
+Wire Wire Line
+	1000 3300 1400 3300
+Connection ~ 2800 3400
+Wire Wire Line
+	2800 3400 2300 3400
+Connection ~ 2800 3700
+Wire Wire Line
+	2800 3700 2300 3700
 $EndSCHEMATC
