File: SuperPower-uC/lowcost/charger_io.sch (KiCad schematic (older format))
At the start: 16 parts, among them J3 USB_C_Receptacle_USB2.0, J4 Solar in, Q3 S8050, Q4 S8050, U5 CH340G, U6 AMS1117-3.3, Y1 12MHZ

Commit message: swapped usb connector back to micro b, testpoints and other stuff
Parts:
- removed J3: USB_C_Receptacle_USB2.0, Connector_USB:USB_C_Receptacle_Palconn_UTC16-G, symbol Connector:USB_C_Receptacle_USB2.0
- removed R19, R20: 5.1k, Resistor_SMD:R_0603_1608Metric_Pad1.05x0.95mm_HandSolder, symbol Device:R
- added J3: USB_B_Micro, Connector_USB:USB_Micro-B_Molex-105017-0001, symbol Connector:USB_B_Micro
- added TP1, TP2: TestPoint, TestPoint:TestPoint_Pad_1.5x1.5mm, symbol Connector:TestPoint
Connections:
- wire segments 64 -> 63
- no-connect marks 8 -> 7
Other:
- moved on the sheet: C5, U6
Changed lines of the file:
@@
 NoConn ~ 7850 3300
 NoConn ~ 7850 3400
-NoConn ~ 3600 4100
-NoConn ~ 3600 4200
-Wire Wire Line
-	3600 3600 3600 3500
-Wire Wire Line
-	3600 3800 3600 3700
-Wire Wire Line
-	3600 3800 3900 3800
+Wire Wire Line
+	3600 3200 3900 3200
 Wire Wire Line
 	4900 2700 4900 2850
@@
 F 4 "C1653" H 6600 3950 50  0001 C CNN "LCSC"
 	1    6600 3950
-	1    0    0    -1
-$EndComp
-$Comp
-L power:GND #PWR0122
-U 1 1 5F7EBB3E
-P 3000 4550
-F 0 "#PWR0122" H 3000 4300 50  0001 C CNN
-F 1 "GND" H 3005 4377 50  0000 C CNN
-F 2 "" H 3000 4550 50  0001 C CNN
-F 3 "" H 3000 4550 50  0001 C CNN
-	1    3000 4550
-	1    0    0    -1
-$EndComp
-$Comp
-L Device:C C5
-U 1 1 5F7DD8B4
-P 6600 5500
-F 0 "C5" H 6700 5550 50  0000 L CNN
-F 1 "1µF" H 6700 5450 50  0000 L CNN
-F 2 "Capacitor_SMD:C_0603_1608Metric_Pad1.05x0.95mm_HandSolder" H 6638 5350 50  0001 C CNN
-F 3 "~" H 6600 5500 50  0001 C CNN
-F 4 "C15849" H 6600 5500 50  0001 C CNN "LCSC"
-	1    6600 5500
 	1    0    0    -1
 $EndComp
@@
 L AMS1117-3.3:AMS1117-3.3 U6
 U 1 1 5F7CB01B
-P 7100 5300
-F 0 "U6" H 7100 5550 50  0000 C CNN
-F 1 "AMS1117-3.3" H 7100 5450 50  0000 C CNN
-F 2 "Package_TO_SOT_SMD:SOT-223-3_TabPin2" H 7400 5000 50  0001 C CNN
-F 3 "http://www.advanced-monolithic.com/pdf/ds1117.pdf" H 7300 5350 50  0001 C CNN
-F 4 "C6186" H 7100 5300 50  0001 C CNN "LCSC"
-	1    7100 5300
+P 7050 5150
+F 0 "U6" H 7050 5400 50  0000 C CNN
+F 1 "AMS1117-3.3" H 7050 5300 50  0000 C CNN
+F 2 "Package_TO_SOT_SMD:SOT-223-3_TabPin2" H 7350 4850 50  0001 C CNN
+F 3 "http://www.advanced-monolithic.com/pdf/ds1117.pdf" H 7250 5200 50  0001 C CNN
+F 4 "C6186" H 7050 5150 50  0001 C CNN "LCSC"
+	1    7050 5150
 	1    0    0    -1
 $EndComp
@@
 $EndComp
 $Comp
-L Connector:USB_C_Receptacle_USB2.0 J3
-U 1 1 5F80E438
-P 3000 3600
-F 0 "J3" H 3107 4467 50  0000 C CNN
-F 1 "USB_C_Receptacle_USB2.0" H 3107 4376 50  0000 C CNN
-F 2 "Connector_USB:USB_C_Receptacle_Palconn_UTC16-G" H 3150 3600 50  0001 C CNN
-F 3 "https://www.usb.org/sites/default/files/documents/usb_type-c.zip" H 3150 3600 50  0001 C CNN
-F 4 "C319148" H 3000 3600 50  0001 C CNN "LCSC"
-	1    3000 3600
-	1    0    0    -1
-$EndComp
-Connection ~ 3600 3800
-$Comp
-L Device:R R19
-U 1 1 5F81A493
-P 3750 3200
-F 0 "R19" V 3650 3100 50  0000 C CNN
-F 1 "5.1k" V 3650 3300 50  0000 C CNN
-F 2 "Resistor_SMD:R_0603_1608Metric_Pad1.05x0.95mm_HandSolder" V 3680 3200 50  0001 C CNN
-F 3 "~" H 3750 3200 50  0001 C CNN
-F 4 "C23186" V 3750 3200 50  0001 C CNN "LCSC"
-	1    3750 3200
-	0    1    1    0
-$EndComp
-$Comp
-L Device:R R20
-U 1 1 5F81C386
-P 3750 3300
-F 0 "R20" V 3850 3200 50  0000 C CNN
-F 1 "5.1k" V 3850 3400 50  0000 C CNN
-F 2 "Resistor_SMD:R_0603_1608Metric_Pad1.05x0.95mm_HandSolder" V 3680 3300 50  0001 C CNN
-F 3 "~" H 3750 3300 50  0001 C CNN
-F 4 "C23186" V 3750 3300 50  0001 C CNN "LCSC"
-	1    3750 3300
-	0    1    1    0
-$EndComp
-Wire Wire Line
-	3900 3200 3900 3300
-Connection ~ 3900 3300
-$Comp
 L power:GND #PWR0125
 U 1 1 5F8616D9
@@
 	1    0    0    -1
 $EndComp
-Wire Wire Line
-	3600 3000 3900 3000
 Connection ~ 4900 2700
 Wire Wire Line
@@
 Connection ~ 3900 3000
 Wire Wire Line
-	7100 5550 7100 5650
-Wire Wire Line
-	7100 5650 7650 5650
-Text Label 7650 5650 2    50   ~ 0
+	7050 5400 7050 5600
+Text Label 7600 5600 2    50   ~ 0
 3v3FTDI
 Text Label 4300 3000 0    50   ~ 0
 VBUS
-Text Label 7650 5350 2    50   ~ 0
+Text Label 7600 5200 2    50   ~ 0
 VBUS
 Wire Wire Line
-	7450 5350 7650 5350
-Wire Wire Line
-	3000 4500 3000 4550
-NoConn ~ 2700 4500
+	7400 5200 7600 5200
 Wire Wire Line
 	6700 2700 7150 2700
@@
 Wire Wire Line
 	6850 3000 7150 3000
-Wire Wire Line
-	7100 5650 6600 5650
-Connection ~ 7100 5650
-Wire Wire Line
-	6750 5350 6600 5350
-Wire Wire Line
-	6600 5350 6400 5350
-Connection ~ 6600 5350
 $Comp
 L power:GND #PWR0126
 U 1 1 5F8B507C
-P 6400 5350
-F 0 "#PWR0126" H 6400 5100 50  0001 C CNN
-F 1 "GND" H 6405 5177 50  0000 C CNN
-F 2 "" H 6400 5350 50  0001 C CNN
-F 3 "" H 6400 5350 50  0001 C CNN
-	1    6400 5350
+P 6350 5200
+F 0 "#PWR0126" H 6350 4950 50  0001 C CNN
+F 1 "GND" H 6355 5027 50  0000 C CNN
+F 2 "" H 6350 5200 50  0001 C CNN
+F 3 "" H 6350 5200 50  0001 C CNN
+	1    6350 5200
 	1    0    0    -1
 $EndComp
@@
 Wire Wire Line
 	4100 3000 3900 3000
-Wire Wire Line
-	4100 3000 4700 3000
-Wire Wire Line
-	3900 3300 4100 3300
-Connection ~ 4100 3300
 Text Label 8200 2700 2    50   ~ 0
 3v3FTDI
@@
 	7850 2700 8200 2700
 Wire Wire Line
-	3600 3600 3900 3600
-Connection ~ 3600 3600
-Text Label 3900 3800 2    50   ~ 0
+	3600 3300 3900 3300
+Text Label 3900 3200 2    50   ~ 0
 D+
-Text Label 3900 3600 2    50   ~ 0
+Text Label 3900 3300 2    50   ~ 0
 D-
 Text Label 6850 3100 0    50   ~ 0
@@
 Wire Wire Line
 	4400 2700 4900 2700
+Wire Wire Line
+	3300 3600 3300 3650
+$Comp
+L power:GND #PWR0122
+U 1 1 5F7EBB3E
+P 3300 3650
+F 0 "#PWR0122" H 3300 3400 50  0001 C CNN
+F 1 "GND" H 3305 3477 50  0000 C CNN
+F 2 "" H 3300 3650 50  0001 C CNN
+F 3 "" H 3300 3650 50  0001 C CNN
+	1    3300 3650
+	1    0    0    -1
+$EndComp
+$Comp
+L Connector:USB_B_Micro J3
+U 1 1 5F937C28
+P 3300 3200
+F 0 "J3" H 3357 3667 50  0000 C CNN
+F 1 "USB_B_Micro" H 3357 3576 50  0000 C CNN
+F 2 "Connector_USB:USB_Micro-B_Molex-105017-0001" H 3357 3575 50  0001 C CNN
+F 3 "https://datasheet.lcsc.com/szlcsc/2002271812_XKB-Connectivity-U254-051T-4BH23-S2B_C319164.pdf" H 3450 3150 50  0001 C CNN
+F 4 "C319164" H 3300 3200 50  0001 C CNN "LCSC"
+	1    3300 3200
+	1    0    0    -1
+$EndComp
+Wire Wire Line
+	3600 3000 3900 3000
+NoConn ~ 3600 3400
+NoConn ~ 3200 3600
+$Comp
+L Connector:TestPoint TP1
+U 1 1 5F960985
+P 7200 5550
+F 0 "TP1" H 7250 5700 50  0000 L CNN
+F 1 "TestPoint" H 7258 5577 50  0001 L CNN
+F 2 "TestPoint:TestPoint_Pad_1.5x1.5mm" H 7400 5550 50  0001 C CNN
+F 3 "~" H 7400 5550 50  0001 C CNN
+	1    7200 5550
+	1    0    0    -1
+$EndComp
+Wire Wire Line
+	6700 5200 6550 5200
+Wire Wire Line
+	6550 5200 6350 5200
+Connection ~ 6550 5200
+$Comp
+L Device:C C5
+U 1 1 5F7DD8B4
+P 6550 5350
+F 0 "C5" H 6650 5400 50  0000 L CNN
+F 1 "1µF" H 6650 5300 50  0000 L CNN
+F 2 "Capacitor_SMD:C_0603_1608Metric_Pad1.05x0.95mm_HandSolder" H 6588 5200 50  0001 C CNN
+F 3 "~" H 6550 5350 50  0001 C CNN
+F 4 "C15849" H 6550 5350 50  0001 C CNN "LCSC"
+	1    6550 5350
+	1    0    0    -1
+$EndComp
+Wire Wire Line
+	6550 5500 6550 5600
+Wire Wire Line
+	6550 5600 7050 5600
+Connection ~ 7050 5600
+Wire Wire Line
+	7050 5600 7200 5600
+Wire Wire Line
+	7200 5550 7200 5600
+Connection ~ 7200 5600
+Wire Wire Line
+	7200 5600 7600 5600
+$Comp
+L Connector:TestPoint TP2
+U 1 1 5F973D21
+P 5350 2700
+F 0 "TP2" H 5400 2850 50  0000 L CNN
+F 1 "TestPoint" H 5408 2727 50  0001 L CNN
+F 2 "TestPoint:TestPoint_Pad_1.5x1.5mm" H 5550 2700 50  0001 C CNN
+F 3 "~" H 5550 2700 50  0001 C CNN
+	1    5350 2700
+	1    0    0    -1
+$EndComp
+Wire Wire Line
+	4100 3000 4700 3000
 $EndSCHEMATC

Commit message: swapped pins for regulator and some more testpoints
Parts:
- added TP6, TP7: TestPoint, TestPoint:TestPoint_Pad_1.5x1.5mm, symbol Connector:TestPoint
Connections:
- wire segments 63 -> 65
Changed lines of the file:
@@
 Connection ~ 8400 2900
 Wire Wire Line
-	8400 2900 7850 2900
+	8400 2900 8100 2900
 Wire Wire Line
 	8350 3000 8350 3250
 Connection ~ 8350 3000
-Wire Wire Line
-	8350 3000 7850 3000
 Wire Wire Line
 	8400 3000 8400 2900
@@
 Wire Wire Line
 	4100 3000 4700 3000
+$Comp
+L Connector:TestPoint TP6
+U 1 1 5F9E682C
+P 8100 2900
+F 0 "TP6" H 8150 3000 50  0000 L CNN
+F 1 "TestPoint" H 8158 2927 50  0001 L CNN
+F 2 "TestPoint:TestPoint_Pad_1.5x1.5mm" H 8300 2900 50  0001 C CNN
+F 3 "~" H 8300 2900 50  0001 C CNN
+	1    8100 2900
+	1    0    0    -1
+$EndComp
+Connection ~ 8100 2900
+Wire Wire Line
+	8100 2900 7850 2900
+$Comp
+L Connector:TestPoint TP7
+U 1 1 5F9ED833
+P 8100 3000
+F 0 "TP7" H 8050 3200 50  0000 L CNN
+F 1 "TestPoint" H 8158 3027 50  0001 L CNN
+F 2 "TestPoint:TestPoint_Pad_1.5x1.5mm" H 8300 3000 50  0001 C CNN
+F 3 "~" H 8300 3000 50  0001 C CNN
+	1    8100 3000
+	-1   0    0    1
+$EndComp
+Connection ~ 8100 3000
+Wire Wire Line
+	8100 3000 7850 3000
+Wire Wire Line
+	8100 3000 8350 3000
 $EndSCHEMATC

Commit message: removed charge led and pcb stuff
Parts:
- removed TP2: TestPoint, TestPoint:TestPoint_Pad_1.5x1.5mm, symbol Connector:TestPoint
Connections:
- wire segments 65 -> 66
- no-connect marks 7 -> 6
Changed lines of the file:
@@
 	3600 3000 3900 3000
 NoConn ~ 3600 3400
-NoConn ~ 3200 3600
 $Comp
 L Connector:TestPoint TP1
@@
 Wire Wire Line
 	7200 5600 7600 5600
-$Comp
-L Connector:TestPoint TP2
-U 1 1 5F973D21
-P 5350 2700
-F 0 "TP2" H 5400 2850 50  0000 L CNN
-F 1 "TestPoint" H 5408 2727 50  0001 L CNN
-F 2 "TestPoint:TestPoint_Pad_1.5x1.5mm" H 5550 2700 50  0001 C CNN
-F 3 "~" H 5550 2700 50  0001 C CNN
-	1    5350 2700
-	1    0    0    -1
-$EndComp
 Wire Wire Line
 	4100 3000 4700 3000
@@
 Wire Wire Line
 	8100 3000 8350 3000
+Wire Wire Line
+	3200 3600 3300 3600
+Connection ~ 3300 3600
 $EndSCHEMATC

Commit message: fixed erc errors
Connections:
- wire segments 66 -> 65
Changed lines of the file:
@@
-$EndComp
-$Comp
-L power:PWR_FLAG #FLG0101
-U 1 1 5F872CCA
-P 3900 3000
-F 0 "#FLG0101" H 3900 3075 50  0001 C CNN
-F 1 "PWR_FLAG" H 3900 3173 50  0000 C CNN
-F 2 "" H 3900 3000 50  0001 C CNN
-F 3 "~" H 3900 3000 50  0001 C CNN
-	1    3900 3000
-	1    0    0    -1
 $EndComp
 $Comp
@@
 	-1   0    0    1
 $EndComp
-Connection ~ 3900 3000
 Wire Wire Line
 	7050 5400 7050 5600
@@
 $EndComp
 Connection ~ 4100 3000
-Wire Wire Line
-	4100 3000 3900 3000
 Text Label 8200 2700 2    50   ~ 0
 3v3FTDI
@@
 	1    0    0    -1
 $EndComp
-Wire Wire Line
-	3600 3000 3900 3000
 NoConn ~ 3600 3400
 $Comp
@@
 	3200 3600 3300 3600
 Connection ~ 3300 3600
+Wire Wire Line
+	3600 3000 4100 3000
 $EndSCHEMATC

Commit message: some minor improvements and disconnected shield
Connections:
- wire segments 65 -> 64
- no-connect marks 6 -> 7
Changed lines of the file:
@@
 	8100 3000 8350 3000
 Wire Wire Line
-	3200 3600 3300 3600
-Connection ~ 3300 3600
-Wire Wire Line
 	3600 3000 4100 3000
+NoConn ~ 3200 3600
 $EndSCHEMATC

Commit message: fixed auto reset transistor footprints
Parts:
- removed Q3, Q4: S8050, Package_TO_SOT_SMD:SOT-23_Handsoldering, symbol Transistor_BJT:S8050
- added Q3, Q4: S8050, Package_TO_SOT_SMD:SOT-23_Handsoldering, symbol Transistor_BJT:BC817
Changed lines of the file:
@@
-$EndComp
-$Comp
-L Transistor_BJT:S8050 Q4
-U 1 1 5F7D2269
-P 9000 3250
-F 0 "Q4" H 9190 3204 50  0000 L CNN
-F 1 "S8050" H 9190 3295 50  0000 L CNN
-F 2 "Package_TO_SOT_SMD:SOT-23_Handsoldering" H 9200 3175 50  0001 L CIN
-F 3 "http://www.unisonic.com.tw/datasheet/S8050.pdf" H 9000 3250 50  0001 L CNN
-F 4 "C111272" H 9000 3250 50  0001 C CNN "LCSC"
-	1    9000 3250
-	1    0    0    1
-$EndComp
-$Comp
-L Transistor_BJT:S8050 Q3
-U 1 1 5F7D1CC7
-P 9000 2700
-F 0 "Q3" H 9190 2746 50  0000 L CNN
-F 1 "S8050" H 9190 2655 50  0000 L CNN
-F 2 "Package_TO_SOT_SMD:SOT-23_Handsoldering" H 9200 2625 50  0001 L CIN
-F 3 "http://www.unisonic.com.tw/datasheet/S8050.pdf" H 9000 2700 50  0001 L CNN
-F 4 "C111272" H 9000 2700 50  0001 C CNN "LCSC"
-	1    9000 2700
-	1    0    0    -1
 $EndComp
 $Comp
@@
 	3600 3000 4100 3000
 NoConn ~ 3200 3600
+$Comp
+L Transistor_BJT:BC817 Q3
+U 1 1 5FC9B8EE
+P 9000 2700
+F 0 "Q3" H 9190 2746 50  0000 L CNN
+F 1 "S8050" H 9190 2655 50  0000 L CNN
+F 2 "Package_TO_SOT_SMD:SOT-23_Handsoldering" H 9200 2625 50  0001 L CIN
+F 3 "https://datasheet.lcsc.com/szlcsc/1811131731_Shikues-S8050_C111272.pdf" H 9000 2700 50  0001 L CNN
+F 4 "C111272" H 9000 2700 50  0001 C CNN "LCSC"
+	1    9000 2700
+	1    0    0    -1
+$EndComp
+$Comp
+L Transistor_BJT:BC817 Q4
+U 1 1 5FCA504B
+P 9000 3250
+F 0 "Q4" H 9190 3204 50  0000 L CNN
+F 1 "S8050" H 9190 3295 50  0000 L CNN
+F 2 "Package_TO_SOT_SMD:SOT-23_Handsoldering" H 9200 3175 50  0001 L CIN
+F 3 "https://datasheet.lcsc.com/szlcsc/1811131731_Shikues-S8050_C111272.pdf" H 9000 3250 50  0001 L CNN
+F 4 "C111272" H 9000 3250 50  0001 C CNN "LCSC"
+	1    9000 3250
+	1    0    0    1
+$EndComp
 $EndSCHEMATC

Commit message: added diode for bootup stability
Parts:
- added D5: B5819W, Diode_SMD:D_SOD-123, symbol Device:D_Schottky
Connections:
- wire segments 64 -> 65
Other:
- moved on the sheet: C6, C7, R8, R9, U5, Y1

Commit message: changed 2 part numbers
Parts:
- Q3, Q4: LCSC C111272 -> C2146
Changed lines of the file:
@@
 F 2 "Package_TO_SOT_SMD:SOT-23_Handsoldering" H 9100 2625 50  0001 L CIN
 F 3 "https://datasheet.lcsc.com/szlcsc/1811131731_Shikues-S8050_C111272.pdf" H 8900 2700 50  0001 L CNN
-F 4 "C111272" H 8900 2700 50  0001 C CNN "LCSC"
+F 4 "C2146" H 8900 2700 50  0001 C CNN "LCSC"
 	1    8900 2700
 	1    0    0    -1
@@
 F 2 "Package_TO_SOT_SMD:SOT-23_Handsoldering" H 9100 3175 50  0001 L CIN
 F 3 "https://datasheet.lcsc.com/szlcsc/1811131731_Shikues-S8050_C111272.pdf" H 8900 3250 50  0001 L CNN
-F 4 "C111272" H 8900 3250 50  0001 C CNN "LCSC"
+F 4 "C2146" H 8900 3250 50  0001 C CNN "LCSC"
 	1    8900 3250
 	1    0    0    1
